File: PocketNode_kicad/display.kicad_sch (KiCad schematic)
At the start: 3 parts, among them J2 display

Commit message: update
Parts:
- C9: footprint (none) -> Capacitor_SMD:C_0603_1608Metric_Pad1.08x0.95mm_HandSolder
- J2: footprint (none) -> Connector_PinHeader_2.54mm:PinHeader_1x07_P2.54mm_Vertical
- R8: footprint (none) -> Resistor_SMD:R_0603_1608Metric_Pad0.98x0.95mm_HandSolder
Changed lines of the file:
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@@
 			)
 		)
-		(property "Footprint" ""
+		(property "Footprint" "Connector_PinHeader_2.54mm:PinHeader_1x07_P2.54mm_Vertical"
 			(at 177.8 76.2 0)
 			(effects
@@
 			)
 		)
-		(property "Footprint" ""
+		(property "Footprint" "Resistor_SMD:R_0603_1608Metric_Pad0.98x0.95mm_HandSolder"
 			(at 156.21 83.82 0)
 			(effects
@@
 			)
 		)
-		(property "Footprint" ""
+		(property "Footprint" "Capacitor_SMD:C_0603_1608Metric_Pad1.08x0.95mm_HandSolder"
 			(at 153.67 68.58 0)
 			(effects

Commit message: update
Parts:
- removed J2: display, Connector_PinHeader_2.54mm:PinHeader_1x07_P2.54mm_Vertical, symbol Connector_Generic_MountingPin:Conn_01x07_MountingPin
- added J3: display, Connector_PinSocket_2.54mm:PinSocket_1x07_P2.54mm_Vertical, symbol Connector_Generic:Conn_01x07
Connections:
- net +3.3V: now also J3.2 (Pin_2)
- net GND: now also J3.1 (Pin_1)
- net LCD_DC: now also J3.6 (Pin_6)
- net LCD_RES: now also J3.5 (Pin_5)
- net SCL: now also J3.3 (Pin_3)
- net SDA: now also J3.4 (Pin_4)
- net at R8.2: now also J3.7 (Pin_7)
Changed lines of the file:
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@@
 	)
 	(symbol
-		(lib_id "Connector_Generic_MountingPin:Conn_01x07_MountingPin")
+		(lib_id "Connector_Generic:Conn_01x07")
 		(at 177.8 76.2 0)
 		(unit 1)
@@
 		(dnp no)
 		(fields_autoplaced yes)
-		(property "Reference" "J2"
-			(at 180.34 75.2855 0)
+		(property "Reference" "J3"
+			(at 180.34 74.9299 0)
 			(effects
 				(font
@@
 		)
 		(property "Value" "display"
-			(at 180.34 77.8255 0)
+			(at 180.34 77.4699 0)
 			(effects
 				(font
@@
 			)
 		)
-		(property "Footprint" "Connector_PinHeader_2.54mm:PinHeader_1x07_P2.54mm_Vertical"
+		(property "Footprint" "Connector_PinSocket_2.54mm:PinSocket_1x07_P2.54mm_Vertical"
 			(at 177.8 76.2 0)
 			(effects
@@
 			)
 		)
-		(property "Description" "Generic connectable mounting pin connector, single row, 01x07, script generated (kicad-library-utils/schlib/autogen/connector/)"
+		(property "Description" "Generic connector, single row, 01x07, script generated (kicad-library-utils/schlib/autogen/connector/)"
 			(at 177.8 76.2 0)
 			(effects
@@
 			)
 		)
-		(pin "1"
-		)
 		(pin "2"
 		)
 		(pin "4"
 		)
-		(pin "7"
+		(pin "6"
+		)
+		(pin "3"
 		)
 		(pin "5"
 		)
-		(pin "MP"
+		(pin "7"
 		)
-		(pin "3"
-		)
-		(pin "6"
+		(pin "1"
 		)
 		(instances
 			(project ""
 				(path "/e2b3b76c-15d2-45d4-9847-56ef7109e38b/c058e23a-95ff-46ea-890f-afb329646003"
-					(reference "J2")
+					(reference "J3")
 					(unit 1)
 				)
