File: PocketNode_kicad/MCU.kicad_sch (KiCad schematic)
At the start: 1 part, among them U3 ESP32-S3-WROOM-1-N16R8

Commit message: update2
Parts:
- added C6, C7: 0.1μF, symbol Device:C_Small
- added R6, R7: 10kΩ, symbol Device:R_Small
- added SW2: SW_RST, symbol Switch:SW_Push
- added SW3: SW_BOOT, symbol Switch:SW_Push
Connections:
- net GND: now reaches U3.1 (GND)
- net GND: now also U3.40 (GND), U3.41 (GND), U3.46 (GND), U3.47 (GND), U3.48 (GND), U3.49 (GND), C6.2, C7.2, SW2.2, SW3.2
- net USB_DM_PROT: now reaches U3.19 (IO11)
- net +3.3V: now reaches U3.2 (3V3)
- net +3.3V: now also C7.1, R6.2, R7.1
- net USB_DP_PROT: now reaches U3.20 (IO12)
- net at U3.27 (IO0): now also R7.2, SW3.1
- net at U3.3 (EN): now also C6.1, R6.1, SW2.1
Other:
- moved on the sheet: U3

Commit message: update3
Parts:
- added C8: 10μF, symbol Device:C_Small
- U3: footprint ESP32-S3-WROOM-1_EXP -> Library:ESP32-S3-WROOM-1_EXP
Connections:
- net +3.3V: now also C8.1
- net GND: now also C8.2
- net LCD_DC: now reaches U3.11 (IO18)
- net LCD_RES: now reaches U3.17 (IO9)
- net LCD_BLK: now reaches U3.18 (IO10)
- net SDA: now reaches U3.21 (IO13)
- net SCL: now reaches U3.22 (IO14)
- net I2S_BCLK: now reaches U3.5 (IO5)
- net I2S_LRCK: now reaches U3.6 (IO6)
- net I2S_DOUT: now reaches U3.7 (IO7)
Other:
- moved on the sheet: C6, C7, R6, R7, SW2, SW3, U3

Commit message: update4
Connections:
- net LCD_DC: now also U3.19 (IO11); no longer U3.11 (IO18)
- net USB_DM_PROT: now also U3.13 (IO19); no longer U3.19 (IO11)
- net USB_DP_PROT: now also U3.14 (IO20); no longer U3.20 (IO12)
- net SD_CD: now reaches U3.23 (IO21)
- net SD_CLK: now reaches U3.28 (IO35)
- net SD_CMD: now reaches U3.29 (IO36)
- net SD_DAT0: now reaches U3.30 (IO37)
- net SD_DAT1: now reaches U3.31 (IO38)
- net SD_DAT2: now reaches U3.32 (IO39)
- net SD_DAT3: now reaches U3.33 (IO40)
- net OPT_CS: now reaches U3.8 (IO15)
- new net OPT_MISO: U3.20 (IO12)
Changed lines of the file:
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@@
-	(wire
-		(pts
-			(xy 96.52 74.93) (xy 128.27 74.93)
-		)
-		(stroke
-			(width 0)
-			(type default)
-		)
-	)
 	(wire
 		(pts
@@
 	(wire
 		(pts
-			(xy 96.52 77.47) (xy 128.27 77.47)
-		)
-		(stroke
-			(width 0)
-			(type default)
-		)
-	)
-	(wire
-		(pts
 			(xy 100.33 20.32) (xy 100.33 24.13)
 		)
@@
 		)
 	)
+	(global_label "SD_CD"
+		(shape input)
+		(at 128.27 85.09 180)
+		(fields_autoplaced yes)
+		(effects
+			(font
+				(size 1.27 1.27)
+			)
+			(justify right)
+		)
+		(property "Intersheetrefs" "${INTERSHEET_REFS}"
+			(at 119.2977 85.09 0)
+			(effects
+				(font
+					(size 1.27 1.27)
+				)
+				(justify right)
+				(hide yes)
+			)
+		)
+	)
+	(global_label "SD_CMD"
+		(shape input)
+		(at 168.91 80.01 0)
+		(fields_autoplaced yes)
+		(effects
+			(font
+				(size 1.27 1.27)
+			)
+			(justify left)
+		)
+		(property "Intersheetrefs" "${INTERSHEET_REFS}"
+			(at 179.3337 80.01 0)
+			(effects
+				(font
+					(size 1.27 1.27)
+				)
+				(justify left)
+				(hide yes)
+			)
+		)
+	)
+	(global_label "SD_CLK"
+		(shape input)
+		(at 168.91 82.55 0)
+		(fields_autoplaced yes)
+		(effects
+			(font
+				(size 1.27 1.27)
+			)
+			(justify left)
+		)
+		(property "Intersheetrefs" "${INTERSHEET_REFS}"
+			(at 178.9104 82.55 0)
+			(effects
+				(font
+					(size 1.27 1.27)
+				)
+				(justify left)
+				(hide yes)
+			)
+		)
+	)
 	(global_label "+3.3V"
 		(shape input)
@@
 		)
 	)
+	(global_label "SD_DAT3"
+		(shape input)
+		(at 168.91 69.85 0)
+		(fields_autoplaced yes)
+		(effects
+			(font
+				(size 1.27 1.27)
+			)
+			(justify left)
+		)
+		(property "Intersheetrefs" "${INTERSHEET_REFS}"
+			(at 179.878 69.85 0)
+			(effects
+				(font
+					(size 1.27 1.27)
+				)
+				(justify left)
+				(hide yes)
+			)
+		)
+	)
+	(global_label "OPT_MISO"
+		(shape input)
+		(at 128.27 77.47 180)
+		(fields_autoplaced yes)
+		(effects
+			(font
+				(size 1.27 1.27)
+			)
+			(justify right)
+		)
+		(property "Intersheetrefs" "${INTERSHEET_REFS}"
+			(at 116.1529 77.47 0)
+			(effects
+				(font
+					(size 1.27 1.27)
+				)
+				(justify right)
+				(hide yes)
+			)
+		)
+	)
+	(global_label "SD_DAT2"
+		(shape input)
+		(at 168.91 72.39 0)
+		(fields_autoplaced yes)
+		(effects
+			(font
+				(size 1.27 1.27)
+			)
+			(justify left)
+		)
+		(property "Intersheetrefs" "${INTERSHEET_REFS}"
+			(at 179.878 72.39 0)
+			(effects
+				(font
+					(size 1.27 1.27)
+				)
+				(justify left)
+				(hide yes)
+			)
+		)
+	)
+	(global_label "OPT_CS"
+		(shape input)
+		(at 128.27 46.99 180)
+		(fields_autoplaced yes)
+		(effects
+			(font
+				(size 1.27 1.27)
+			)
+			(justify right)
+		)
+		(property "Intersheetrefs" "${INTERSHEET_REFS}"
+			(at 118.2696 46.99 0)
+			(effects
+				(font
+					(size 1.27 1.27)
+				)
+				(justify right)
+				(hide yes)
+			)
+		)
+	)
+	(global_label "SD_DAT1"
+		(shape input)
+		(at 168.91 74.93 0)
+		(fields_autoplaced yes)
+		(effects
+			(font
+				(size 1.27 1.27)
+			)
+			(justify left)
+		)
+		(property "Intersheetrefs" "${INTERSHEET_REFS}"
+			(at 179.878 74.93 0)
+			(effects
+				(font
+					(size 1.27 1.27)
+				)
+				(justify left)
+				(hide yes)
+			)
+		)
+	)
 	(global_label "I2S_BCLK"
 		(shape input)
@@
 	(global_label "LCD_DC"
 		(shape input)
-		(at 128.27 54.61 180)
-		(fields_autoplaced yes)
-		(effects
-			(font
-				(size 1.27 1.27)
-			)
-			(justify right)
-		)
-		(property "Intersheetrefs" "${INTERSHEET_REFS}"
-			(at 118.2091 54.61 0)
+		(at 128.27 74.93 180)
+		(fields_autoplaced yes)
+		(effects
+			(font
+				(size 1.27 1.27)
+			)
+			(justify right)
+		)
+		(property "Intersheetrefs" "${INTERSHEET_REFS}"
+			(at 118.2091 74.93 0)
 			(effects
 				(font
@@
 		)
 	)
+	(global_label "SD_DAT0"
+		(shape input)
+		(at 168.91 77.47 0)
+		(fields_autoplaced yes)
+		(effects
+			(font
+				(size 1.27 1.27)
+			)
+			(justify left)
+		)
+		(property "Intersheetrefs" "${INTERSHEET_REFS}"
+			(at 179.878 77.47 0)
+			(effects
+				(font
+					(size 1.27 1.27)
+				)
+				(justify left)
+				(hide yes)
+			)
+		)
+	)
 	(global_label "SDA"
 		(shape input)
@@
 	(global_label "USB_DM_PROT"
 		(shape input)
-		(at 96.52 74.93 180)
-		(fields_autoplaced yes)
-		(effects
-			(font
-				(size 1.27 1.27)
-			)
-			(justify right)
-		)
-		(property "Intersheetrefs" "${INTERSHEET_REFS}"
-			(at 80.2301 74.93 0)
+		(at 128.27 59.69 180)
+		(fields_autoplaced yes)
+		(effects
+			(font
+				(size 1.27 1.27)
+			)
+			(justify right)
+		)
+		(property "Intersheetrefs" "${INTERSHEET_REFS}"
+			(at 111.9801 59.69 0)
 			(effects
 				(font
@@
 	(global_label "USB_DP_PROT"
 		(shape input)
-		(at 96.52 77.47 180)
-		(fields_autoplaced yes)
-		(effects
-			(font
-				(size 1.27 1.27)
-			)
-			(justify right)
-		)
-		(property "Intersheetrefs" "${INTERSHEET_REFS}"
-			(at 80.4115 77.47 0)
-			(effects
-				(font
+		(at 128.27 62.23 180)
+		(fields_autoplaced yes)
+		(effects
+			(font
+				(size 1.27 1.27)
+			)
+			(justify right)
+		)
+		(property "Intersheetrefs" "${INTERSHEET_REFS}"
+			(at 112.1615 62.23 0)
+			(effects
+				(font

Commit message: update5
Connections:
- net BTN_1: now reaches U3.10 (IO17)
- net BTN_3: now reaches U3.12 (IO8)
- net ENC_SW: now reaches U3.15 (IO3)
- net ENC_B: now reaches U3.38 (IO2)
- net ENC_A: now reaches U3.39 (IO1)
- net LED: now reaches U3.4 (IO4)
- net BTN_2: now reaches U3.9 (IO16)
- no-connect marks 0 -> 9
Changed lines of the file:
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@@
 		(color 0 0 0 0)
 	)
+	(no_connect
+		(at 128.27 67.31)
+	)
+	(no_connect
+		(at 168.91 87.63)
+	)
+	(no_connect
+		(at 168.91 64.77)
+	)
+	(no_connect
+		(at 168.91 90.17)
+	)
+	(no_connect
+		(at 168.91 67.31)
+	)
+	(no_connect
+		(at 128.27 54.61)
+	)
+	(no_connect
+		(at 168.91 59.69)
+	)
+	(no_connect
+		(at 168.91 62.23)
+	)
+	(no_connect
+		(at 128.27 87.63)
+	)
 	(wire
 		(pts
@@
 		)
 	)
+	(global_label "BTN_1"
+		(shape input)
+		(at 128.27 52.07 180)
+		(fields_autoplaced yes)
+		(effects
+			(font
+				(size 1.27 1.27)
+			)
+			(justify right)
+		)
+		(property "Intersheetrefs" "${INTERSHEET_REFS}"
+			(at 119.5396 52.07 0)
+			(effects
+				(font
+					(size 1.27 1.27)
+				)
+				(justify right)
+				(hide yes)
+			)
+		)
+	)
 	(global_label "SD_DAT3"
 		(shape input)
@@
 		)
 	)
+	(global_label "ENC_A"
+		(shape input)
+		(at 168.91 54.61 0)
+		(fields_autoplaced yes)
+		(effects
+			(font
+				(size 1.27 1.27)
+			)
+			(justify left)
+		)
+		(property "Intersheetrefs" "${INTERSHEET_REFS}"
+			(at 177.7009 54.61 0)
+			(effects
+				(font
+					(size 1.27 1.27)
+				)
+				(justify left)
+				(hide yes)
+			)
+		)
+	)
 	(global_label "SD_DAT2"
 		(shape input)
@@
 		)
 	)
+	(global_label "ENC_B"
+		(shape input)
+		(at 168.91 57.15 0)
+		(fields_autoplaced yes)
+		(effects
+			(font
+				(size 1.27 1.27)
+			)
+			(justify left)
+		)
+		(property "Intersheetrefs" "${INTERSHEET_REFS}"
+			(at 177.8823 57.15 0)
+			(effects
+				(font
+					(size 1.27 1.27)
+				)
+				(justify left)
+				(hide yes)
+			)
+		)
+	)
 	(global_label "LCD_DC"
 		(shape input)
@@
 		)
 	)
+	(global_label "BTN_3"
+		(shape input)
+		(at 128.27 57.15 180)
+		(fields_autoplaced yes)
+		(effects
+			(font
+				(size 1.27 1.27)
+			)
+			(justify right)
+		)
+		(property "Intersheetrefs" "${INTERSHEET_REFS}"
+			(at 119.5396 57.15 0)
+			(effects
+				(font
+					(size 1.27 1.27)
+				)
+				(justify right)
+				(hide yes)
+			)
+		)
+	)
 	(global_label "LCD_BLK"
 		(shape input)
@@
 		)
 	)
+	(global_label "BTN_2"
+		(shape input)
+		(at 128.27 49.53 180)
+		(fields_autoplaced yes)
+		(effects
+			(font
+				(size 1.27 1.27)
+			)
+			(justify right)
+		)
+		(property "Intersheetrefs" "${INTERSHEET_REFS}"
+			(at 119.5396 49.53 0)
+			(effects
+				(font
+					(size 1.27 1.27)
+				)
+				(justify right)
+				(hide yes)
+			)
+		)
+	)
+	(global_label "ENC_SW"
+		(shape input)
+		(at 128.27 64.77 180)
+		(fields_autoplaced yes)
+		(effects
+			(font
+				(size 1.27 1.27)
+			)
+			(justify right)
+		)
+		(property "Intersheetrefs" "${INTERSHEET_REFS}"
+			(at 117.9068 64.77 0)
+			(effects
+				(font
+					(size 1.27 1.27)
+				)
+				(justify right)
+				(hide yes)
+			)
+		)
+	)
 	(global_label "I2S_DOUT"
 		(shape input)
@@
 			(effects
 				(font
+					(size 1.27 1.27)
+				)
+				(justify right)
+				(hide yes)
+			)
+		)
+	)
+	(global_label "LED"
+		(shape input)
+		(at 128.27 36.83 180)
+		(fields_autoplaced yes)
+		(effects
+			(font
+				(size 1.27 1.27)
+			)
+			(justify right)
+		)
+		(property "Intersheetrefs" "${INTERSHEET_REFS}"
+			(at 121.8377 36.83 0)
+			(effects
+				(font

Commit message: update
Parts:
- C6, C7, C8: footprint (none) -> Capacitor_SMD:C_0603_1608Metric_Pad1.08x0.95mm_HandSolder
- R6, R7: footprint (none) -> Resistor_SMD:R_0603_1608Metric_Pad0.98x0.95mm_HandSolder
Changed lines of the file:
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@@
 			)
 		)
-		(property "Footprint" ""
+		(property "Footprint" "Resistor_SMD:R_0603_1608Metric_Pad0.98x0.95mm_HandSolder"
 			(at 76.2 34.29 0)
 			(effects
@@
 			)
 		)
-		(property "Footprint" ""
+		(property "Footprint" "Resistor_SMD:R_0603_1608Metric_Pad0.98x0.95mm_HandSolder"
 			(at 199.39 85.09 0)
 			(effects
@@
 			)
 		)
-		(property "Footprint" ""
+		(property "Footprint" "Capacitor_SMD:C_0603_1608Metric_Pad1.08x0.95mm_HandSolder"
 			(at 83.82 39.37 0)
 			(effects
@@
 			)
 		)
-		(property "Footprint" ""
+		(property "Footprint" "Capacitor_SMD:C_0603_1608Metric_Pad1.08x0.95mm_HandSolder"
 			(at 100.33 26.67 0)
 			(effects
@@
 			)
 		)
-		(property "Footprint" ""
+		(property "Footprint" "Capacitor_SMD:C_0603_1608Metric_Pad1.08x0.95mm_HandSolder"
 			(at 90.17 26.67 0)
 			(effects

Commit message: update
Parts:
- removed SW2: SW_RST, symbol Switch:SW_Push
- removed SW3: SW_BOOT, symbol Switch:SW_Push
- added S1: SW_BOOT, Library:SW_SKRPACE010, symbol Library:SKRPACE010
- added S2: SW_RST, Library:SW_SKRPACE010, symbol Library:SKRPACE010
Connections:
- net GND: now also S1.3, S1.4, S2.3, S2.4
- net at C6.1, R6.1, U3.3 (EN): now also S2.1, S2.2
- net at R7.2, U3.27 (IO0): now also S1.1, S1.2

Commit message: update11
Parts:
- added R26, R27: 100kΩ, Resistor_SMD:R_0603_1608Metric_Pad0.98x0.95mm_HandSolder, symbol Device:R_Small
Connections:
- net BTN_3: now also U3.11 (IO18); no longer U3.12 (IO8)
- net GND: now also R27.1
- new net: R26.1, R27.2, U3.12 (IO8)
- new net VBAT: R26.2
- no-connect marks 9 -> 8

Commit message: s
Parts:
- added C38: 0.1μF, Capacitor_SMD:C_0603_1608Metric_Pad1.08x0.95mm_HandSolder, symbol Device:C_Small
Connections:
- net GND: now also C38.2
- net at R7.2, S1.1, S1.2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: now also C38.1
Changed lines of the file:
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@@
+	)
+	(junction
+		(at 196.85 85.09)
+		(diameter 0)
+		(color 0 0 0 0)
 	)
 	(junction
@@
 	(wire
 		(pts
+			(xy 196.85 85.09) (xy 196.85 87.63)
+		)
+		(stroke
+			(width 0)
+			(type default)
+		)
+	)
+	(wire
+		(pts
 			(xy 193.04 93.98) (xy 193.04 96.52)
 		)
@@
 		(pts
 			(xy 168.91 49.53) (xy 168.91 52.07)
+		)
+		(stroke
+			(width 0)
+			(type default)
+		)
+	)
+	(wire
+		(pts
+			(xy 196.85 96.52) (xy 196.85 92.71)
 		)
 		(stroke
@@
 	(symbol
 		(lib_id "power:GND")
+		(at 196.85 96.52 0)
+		(unit 1)
+		(exclude_from_sim no)
+		(in_bom yes)
+		(on_board yes)
+		(dnp no)
+		(fields_autoplaced yes)
+		(property "Reference" "#PWR075"
+			(at 196.85 102.87 0)
+			(effects
+				(font
+					(size 1.27 1.27)
+				)
+				(hide yes)
+			)
+		)
+		(property "Value" "GND"
+			(at 196.85 101.6 0)
+			(effects
+				(font
+					(size 1.27 1.27)
+				)
+			)
+		)
+		(property "Footprint" ""
+			(at 196.85 96.52 0)
+			(effects
+				(font
+					(size 1.27 1.27)
+				)
+				(hide yes)
+			)
+		)
+		(property "Datasheet" ""
+			(at 196.85 96.52 0)
+			(effects
+				(font
+					(size 1.27 1.27)
+				)
+				(hide yes)
+			)
+		)
+		(property "Description" "Power symbol creates a global label with name \"GND\" , ground"
+			(at 196.85 96.52 0)
+			(effects
+				(font
+					(size 1.27 1.27)
+				)
+				(hide yes)
+			)
+		)
+		(pin "1"
+		)
+		(instances
+			(project "PocketNode"
+				(path "/e2b3b76c-15d2-45d4-9847-56ef7109e38b/c3bd9f70-08e8-4658-b168-675f40b62085"
+					(reference "#PWR075")
+					(unit 1)
+				)
+			)
+		)
+	)
+	(symbol
+		(lib_id "power:GND")
 		(at 128.27 29.21 270)
 		(unit 1)
@@
 					(unit 1)
 				)
+			)
+		)
+	)
+	(symbol
+		(lib_id "Device:C_Small")
+		(at 196.85 90.17 0)
+		(unit 1)
+		(exclude_from_sim no)
+		(in_bom yes)
+		(on_board yes)
+		(dnp no)
+		(fields_autoplaced yes)
+		(property "Reference" "C38"
+			(at 199.39 88.9062 0)
+			(effects
+				(font
+					(size 1.27 1.27)
+				)
+				(justify left)
+			)
+		)
+		(property "Value" "0.1μF"
+			(at 199.39 91.4462 0)
+			(effects
+				(font
+					(size 1.27 1.27)
+				)
+				(justify left)
+			)
+		)
+		(property "Footprint" "Capacitor_SMD:C_0603_1608Metric_Pad1.08x0.95mm_HandSolder"
+			(at 196.85 90.17 0)
+			(effects
+				(font
+					(size 1.27 1.27)
+				)
+				(hide yes)
+			)
+		)
+		(property "Datasheet" "~"
+			(at 196.85 90.17 0)
+			(effects
+				(font
+					(size 1.27 1.27)
+				)
+				(hide yes)
+			)
+		)
+		(property "Description" "Unpolarized capacitor, small symbol"
+			(at 196.85 90.17 0)
+			(effects
+				(font
+					(size 1.27 1.27)
+				)
+				(hide yes)
+			)
+		)
+		(pin "1"
+		)
+		(pin "2"
+		)
+		(instances
+			(project "PocketNode"
+				(path "/e2b3b76c-15d2-45d4-9847-56ef7109e38b/c3bd9f70-08e8-4658-b168-675f40b62085"
+					(reference "C38")
+					(unit 1)
+				)
