File: PocketNode_kicad/PocketNode.kicad_pcb (KiCad board)
At the start: 2 copper layers, 48 x 58 mm, 94 parts, among them J1 USB4105-GF-A, J3 display, J4 MJ-8435, J5 DM3AT-SF-PEJM5, Q1 MMBT3904, SW1 Power, SW4 ENC_SW, SW5 SW1, SW6 SW2, SW7 SW3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

Commit message: s
Parts:
- added C38: 0.1μF, Capacitor_SMD:C_0603_1608Metric_Pad1.08x0.95mm_HandSolder, F.Cu at (126.6, 124.2)
- moved C6 121.2 mm to (193.2, 139.4), turned to -90 degrees
- moved J5 114.6 mm to (164.1, 136.0), turned to 0 degrees
- moved R6 114.3 mm to (190.8, 137.0), turned to 180 degrees
- moved R26 109.9 mm to (192.6, 127.5)
- moved R27 109.6 mm to (192.6, 129.0), turned to 180 degrees
- moved U1 106.8 mm to (199.9, 97.1)
- moved S1 106.2 mm to (115.8, 122.6)
- moved U2 103.3 mm to (193.1, 97.6)
- moved U5 91.4 mm to (201.9, 109.5), turned to -90 degrees
- moved BT1 91.2 mm to (190.6, 102.6), turned to 90 degrees
- moved VR1 77.6 mm to (186.9, 96.3)
- moved S2 77.1 mm to (189.6, 139.6)
- moved J1 76.8 mm to (158.6, 92.1)
- moved U4 69.4 mm to (177.6, 99.3)
- moved R7 46.9 mm to (124.6, 118.1), turned to 180 degrees
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Routing:
- net GND: track 0.00 -> 75.3 mm
- net SD_DAT1: track 0.00 -> 8.56 mm, vias 0 -> 2
- net SD_CMD: track 0.00 -> 7.76 mm, vias 0 -> 2
- net SD_CLK: track 0.00 -> 6.26 mm, vias 0 -> 2
- net SD_DAT2: track 0.00 -> 5.98 mm, vias 0 -> 2
- net SD_DAT0: track 0.00 -> 5.80 mm
Other:
- board size 48 x 58 mm -> 48 x 124.5 mm
