File: PocketNode_kicad/PocketNode.kicad_pcb (KiCad board)
At the start: 2 copper layers, 8.9 x 15.9 mm, 80 parts, among them J1 USB4105-GF-A, J2 display, Q1 MMBT3904, U1 USBLC6-2SC6, U2 MCP73831T-2ACI_OT, U3 ESP32-S3-WROOM-1-N16R8, U4 PCM5102APWR, U5 NJM2073M-ND, U6 PMW3360DM-T2QU, U7 TPS73601DBVR

Commit message: update
Parts:
- added BT1: 502030 LiPo, Connector_PinHeader_2.54mm:PinHeader_1x02_P2.54mm_Vertical, F.Cu at (59.1, 41.1)
- added FB1: 120Ω@100MHz, Library:BEADC1608X95N, F.Cu at (63.4, 40.0)
- added J4: MJ-8435, Library:MJ-8435, F.Cu at (61.3, 23.2)
- added J5: DM3AT-SF-PEJM5, Library:HRS_DM3AT-SF-PEJM5, F.Cu at (42.2, 30.4)
- added R25: 10kΩ, Resistor_SMD:R_0603_1608Metric_Pad0.98x0.95mm_HandSolder, F.Cu at (52.6, 21.4)

Commit message: update
Parts:
- removed J2: display, Connector_PinHeader_2.54mm:PinHeader_1x07_P2.54mm_Vertical
- added J3: display, Connector_PinSocket_2.54mm:PinSocket_1x07_P2.54mm_Vertical, F.Cu at (118.0, 78.3)
- added S1: SW_BOOT, Library:SW_SKRPACE010, F.Cu at (178.0, 46.5)
- added S2: SW_RST, Library:SW_SKRPACE010, F.Cu at (178.0, 51.2)
- added SW1: Power, Button_Switch_THT:SW_Slide_SPDT_Angled_CK_OS102011MA1Q, F.Cu at (149.9, 75.0)
- added SW4: ENC_SW, Button_Switch_THT:SW_Tactile_SPST_Angled_PTS645Vx39-2LFS, F.Cu at (138.0, 61.5)
- added SW5: SW1, Button_Switch_THT:SW_PUSH_6mm, F.Cu at (137.2, 26.6)
- added SW6: SW2, Button_Switch_THT:SW_PUSH_6mm, F.Cu at (137.2, 35.2)
- added SW7: SW3, Button_Switch_THT:SW_PUSH_6mm, F.Cu at (137.2, 43.8)
- moved Q1 157.2 mm to (214.8, 48.0)
- moved U2 157.2 mm to (201.7, 41.5)
- moved U7 157.2 mm to (207.1, 48.0)
- moved U1 157.2 mm to (195.9, 41.5)
- moved VR1 157.2 mm to (207.4, 41.5)
- moved J5 132.0 mm to (174.2, 33.1), turned to 180 degrees
- moved J1 120.4 mm to (158.5, 25.5), turned to 180 degrees
- moved U4 109.5 mm to (150.5, 58.0)
- moved J4 98.0 mm to (141.5, 79.5), turned to 180 degrees
- moved U3 96.8 mm to (170.8, 69.1), turned to 180 degrees
- moved U6 70.0 mm to (158.5, 44.0)
- moved VR2 69.7 mm to (140.1, 54.0)
- moved U5 41.7 mm to (150.5, 68.0)
Other:
- board size 8.9 x 15.9 mm -> 48 x 58 mm

Commit message: update
Parts:
- moved SW1 59.7 mm to (105.6, 35.0)
- moved SW6 21.0 mm to (118.8, 25.2)
- moved SW7 21.0 mm to (118.8, 33.8)
- moved SW5 21.0 mm to (118.8, 16.7)
- moved VR2 15.1 mm to (125.0, 53.0)
Changed lines of the file:
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@@
 	(footprint "Button_Switch_THT:SW_PUSH_6mm"
 		(layer "F.Cu")
-		(at 137.25 35.2)
+		(at 118.75 25.25)
 		(descr "Generic 6mm SW tactile push button")
 		(tags "tact sw push 6mm")
@@
 	(footprint "Button_Switch_THT:SW_Slide_SPDT_Angled_CK_OS102011MA1Q"
 		(layer "F.Cu")
-		(at 149.9 75)
+		(at 105.6 35)
 		(descr "CuK miniature slide switch, OS series, SPDT, right angle, http://www.ckswitches.com/media/1428/os.pdf")
 		(tags "switch SPDT")
@@
 	(footprint "Library:TRIM_EC10E1220501"
 		(layer "F.Cu")
-		(at 140.1 54)
+		(at 125 53)
 		(property "Reference" "VR2"
-			(at -2.828385 -5.641775 0)
+			(at 0 -3 0)
 			(layer "F.SilkS")
 			(effects
@@
 	(footprint "Button_Switch_THT:SW_PUSH_6mm"
 		(layer "F.Cu")
-		(at 137.25 43.75)
+		(at 118.75 33.8)
 		(descr "Generic 6mm SW tactile push button")
 		(tags "tact sw push 6mm")
@@
 	(footprint "Button_Switch_THT:SW_PUSH_6mm"
 		(layer "F.Cu")
-		(at 137.25 26.65)
+		(at 118.75 16.7)
 		(descr "Generic 6mm SW tactile push button")
 		(tags "tact sw push 6mm")

Commit message: update
Parts:
- moved BT1 108.3 mm to (167.2, 48.1)
- moved VR2 57.9 mm to (179.9, 34.7), turned to 90 degrees
- moved U5 31.5 mm to (119.1, 70.9)
- moved U4 30.8 mm to (119.8, 60.8)
- moved J5 27.0 mm to (200.5, 27.3)
- moved J4 12.5 mm to (129.0, 80.3)
- moved U3 12.3 mm to (158.5, 68.9)
- moved SW4 11.2 mm to (126.9, 60.1)
- moved D1 5.60 mm to (105.1, 78.1)
- moved D2 5.60 mm to (105.1, 80.7)
- moved D3 5.60 mm to (105.1, 83.3)
- moved D4 5.60 mm to (105.1, 85.9)
Changed lines of the file:
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@@
 		)
 		(embedded_fonts no)
+		(model "${KIPRJMOD}/lib/MMBT3904/MMBT3904.step"
+			(offset
+				(xyz 0 0 0)
+			)
+			(scale
+				(xyz 1 1 1)
+			)
+			(rotate
+				(xyz -90 -0 -0)
+			)
+		)
 	)
 	(footprint "Resistor_SMD:R_0603_1608Metric_Pad0.98x0.95mm_HandSolder"
@@
 	(footprint "Diode_SMD:D_0603_1608Metric_Pad1.05x0.95mm_HandSolder"
 		(layer "F.Cu")
-		(at 99.535 83.03)
+		(at 105.125 83.28)
 		(descr "Diode SMD 0603 (1608 Metric), square (rectangular) end terminal, IPC-7351 nominal, (Body size source: http://www.tortai-tech.com/upload/download/2011102023233369053.pdf), generated with kicad-footprint-generator")
 		(tags "diode handsolder")
@@
 	(footprint "Button_Switch_THT:SW_Tactile_SPST_Angled_PTS645Vx39-2LFS"
 		(layer "F.Cu")
-		(at 138 61.5)
+		(at 126.925 60.1125)
 		(descr "tactile switch SPST right angle, PTS645VL39-2 LFS")
 		(tags "tactile switch SPST angled PTS645VL39-2 LFS C&K Button")
@@
 		)
 		(embedded_fonts no)
+		(model "${KIPRJMOD}/lib/USB4105-GF-A/USB4105-GF-A.step"
+			(offset
+				(xyz 0 0 0)
+			)
+			(scale
+				(xyz 1 1 1)
+			)
+			(rotate
+				(xyz -90 -0 -0)
+			)
+		)
 	)
 	(footprint "Capacitor_SMD:C_0603_1608Metric_Pad1.08x0.95mm_HandSolder"
@@
 		)
 		(embedded_fonts no)
+		(model "${KIPRJMOD}/lib/TPS73601DBVR/TPS73601DBVR.step"
+			(offset
+				(xyz 0 0 0)
+			)
+			(scale
+				(xyz 1 1 1)
+			)
+			(rotate
+				(xyz -90 -0 -0)
+			)
+		)
 	)
 	(footprint "Resistor_SMD:R_0603_1608Metric_Pad0.98x0.95mm_HandSolder"
@@
 	(footprint "Diode_SMD:D_0603_1608Metric_Pad1.05x0.95mm_HandSolder"
 		(layer "F.Cu")
-		(at 99.535 85.62)
+		(at 105.125 85.87)
 		(descr "Diode SMD 0603 (1608 Metric), square (rectangular) end terminal, IPC-7351 nominal, (Body size source: http://www.tortai-tech.com/upload/download/2011102023233369053.pdf), generated with kicad-footprint-generator")
 		(tags "diode handsolder")
@@
 		)
 		(embedded_fonts no)
+		(model "${KIPRJMOD}/lib/TPS73601DBVR/TPS73601DBVR.step"
+			(offset
+				(xyz 0 0 0)
+			)
+			(scale
+				(xyz 1 1 1)
+			)
+			(rotate
+				(xyz -90 -0 -0)
+			)
+		)
 	)
 	(footprint "Capacitor_SMD:C_0603_1608Metric_Pad1.08x0.95mm_HandSolder"
@@
 	(footprint "Library:NJR-DMP8_NJR"
 		(layer "F.Cu")
-		(at 150.5 68)
+		(at 119.1 70.9)
 		(tags "NJM2073M-ND ")
 		(property "Reference" "U5"
@@
 		(fp_text user "*"
 			(at -2.2225 -2.5781 0)
-			(unlocked yes)
 			(layer "F.Fab")
 			(effects
@@
 	(footprint "LED_SMD:LED_0603_1608Metric_Pad1.05x0.95mm_HandSolder"
 		(layer "F.Cu")
-		(at 99.535 77.85)
+		(at 105.125 78.1)
 		(descr "LED SMD 0603 (1608 Metric), square (rectangular) end terminal, IPC-7351 nominal, (Body size source: http://www.tortai-tech.com/upload/download/2011102023233369053.pdf), generated with kicad-footprint-generator")
 		(tags "LED handsolder")
@@
 	(footprint "Library:TRIM_EC10E1220501"
 		(layer "F.Cu")
-		(at 125 53)
+		(at 179.946 34.7 90)
 		(property "Reference" "VR2"
-			(at 0 -3 0)
+			(at 0 -3 90)
 			(layer "F.SilkS")
 			(effects
@@
 		)
 		(property "Value" "EC10E"
-			(at 4.798145 4.367845 0)
+			(at 4.798145 4.367845 90)
 			(layer "F.Fab")
 			(effects
@@
 		)
 		(property "Datasheet" ""
-			(at 0 0 0)
+			(at 0 0 90)
 			(layer "F.Fab")
 			(hide yes)
@@
 		)
 		(property "Description" ""
-			(at 0 0 0)
+			(at 0 0 90)
 			(layer "F.Fab")
 			(hide yes)
@@
 		(attr through_hole)
 		(pad "" np_thru_hole circle
-			(at -5.4 -2)
+			(at -5.4 -2 90)
 			(size 2 2)
 			(drill 2)
@@
 		)
 		(pad "" np_thru_hole circle
-			(at 5.4 -2)
+			(at 5.4 -2 90)
 			(size 2 2)
 			(drill 2)
@@
 		)
 		(pad "A" thru_hole oval
-			(at -2.5 0)
+			(at -2.5 0 90)
 			(size 1.508 3.016)
 			(drill 1)
@@
 		)
 		(pad "B" thru_hole oval
-			(at 0 0)
+			(at 0 0 90)
 			(size 1.508 3.016)
 			(drill 1)
@@
 		)
 		(pad "C" thru_hole oval
-			(at 2.5 0)
+			(at 2.5 0 90)
 			(size 1.508 3.016)
 			(drill 1)
@@
 	(footprint "Connector_PinHeader_2.54mm:PinHeader_1x02_P2.54mm_Vertical"
 		(layer "F.Cu")
-		(at 59.1 41.06)
+		(at 167.2 48.125)
 		(descr "Through hole straight pin header, 1x02, 2.54mm pitch, single row")
 		(tags "Through hole pin header THT 1x02 2.54mm single row")
@@
 	(footprint "Library:ESP32-S3-WROOM-1_EXP"
 		(layer "F.Cu")
-		(at 170.75 69.13 180)
+		(at 158.5 68.86 180)
 		(tags "ESP32-S3-WROOM-1-N16R8 ")
 		(property "Reference" "U3"
@@
 		(fp_text user "*"
 			(at -7.3657 -5.26 180)
-			(unlocked yes)
 			(layer "F.Fab")
 			(effects
@@
 			(polygon
 				(pts
-					(xy 179.7543 81.8808) (xy 179.7543 75.8864) (xy 161.7457 75.8864) (xy 161.7457 81.8808)
+					(xy 167.5043 81.6108) (xy 167.5043 75.6164) (xy 149.4957 75.6164) (xy 149.4957 81.6108)
 				)
 			)
@@
 	(footprint "Library:HRS_DM3AT-SF-PEJM5"
 		(layer "F.Cu")
-		(at 174.175 33.125 180)
+		(at 200.5 27.3 180)
 		(property "Reference" "J5"
 			(at -4.41177 -12.95097 0)
@@
 			(polygon
 				(pts
-					(xy 171.25 26.4) (xy 168.7 26.4) (xy 168.7 25.05) (xy 171.25 25.05)
+					(xy 197.575 20.575) (xy 195.025 20.575) (xy 195.025 19.225) (xy 197.575 19.225)
 				)
 			)
@@
 			(polygon
 				(pts
-					(xy 179.6 36.1) (xy 170.9 36.1) (xy 170.9 34.5) (xy 179.6 34.5)
+					(xy 205.925 30.275) (xy 197.225 30.275) (xy 197.225 28.675) (xy 205.925 28.675)
 				)
 			)
@@
 			(polygon
 				(pts
-					(xy 180.3 34.8) (xy 179.6 34.8) (xy 179.6 27.2) (xy 180.3 27.2)
+					(xy 206.625 28.975) (xy 205.925 28.975) (xy 205.925 21.375) (xy 206.625 21.375)
 				)
 			)
@@
 			(polygon
 				(pts
-					(xy 181.4 36.2) (xy 180.65 36.2) (xy 180.65 32.6) (xy 181.4 32.6)
+					(xy 207.725 30.375) (xy 206.975 30.375) (xy 206.975 26.775) (xy 207.725 26.775)
 				)
 			)
@@
 			(polygon
 				(pts
-					(xy 181.4 40.65) (xy 180.65 40.65) (xy 180.65 37.4) (xy 181.4 37.4)
+					(xy 207.725 34.825) (xy 206.975 34.825) (xy 206.975 31.575) (xy 207.725 31.575)
 				)
 			)
 		)
 		(embedded_fonts no)
+		(model "${KIPRJMOD}/lib/DM3AT-SF-PEJM5/DM3AT-SF-PEJM5.step"
+			(offset
+				(xyz 0 0 0)
+			)
+			(scale
+				(xyz 1 1 1)
+			)
+			(rotate
+				(xyz -90 -0 -0)
+			)
+		)
 	)
 	(footprint "Capacitor_SMD:C_0805_2012Metric_Pad1.18x1.45mm_HandSolder"
@@
 		)
 		(embedded_fonts no)
+		(model "${KIPRJMOD}/lib/USBLC6-2SC6/USBLC6-2SC6.step"
+			(offset
+				(xyz 0 0 0)
+			)
+			(scale
+				(xyz 1 1 1)
+			)
+			(rotate
+				(xyz -90 -0 -0)
+			)
+		)
 	)
 	(footprint "Capacitor_SMD:C_0603_1608Metric_Pad1.08x0.95mm_HandSolder"
@@
 		)
 		(embedded_fonts no)
+		(model "${KIPRJMOD}/lib/BLM18PG121SN1D/BLM18PG121SN1D.step"
+			(offset
+				(xyz 0 0 0)
+			)
+			(scale
+				(xyz 1 1 1)
+			)
+			(rotate
+				(xyz -90 -0 -0)
+			)
+		)
 	)
 	(footprint "Resistor_SMD:R_0603_1608Metric_Pad0.98x0.95mm_HandSolder"
@@
 		)
 		(embedded_fonts no)
+		(model "${KIPRJMOD}/lib/MMBT3904/MMBT3904.step"
+			(offset
+				(xyz 0 0 0)
+			)
+			(scale
+				(xyz 1 1 1)
+			)
+			(rotate
+				(xyz -90 -0 -0)
+			)
+		)
 	)
 	(footprint "Button_Switch_THT:SW_PUSH_6mm"
@@
 	(footprint "LED_SMD:LED_0603_1608Metric_Pad1.05x0.95mm_HandSolder"
 		(layer "F.Cu")
-		(at 99.535 80.44)
+		(at 105.125 80.69)
 		(descr "LED SMD 0603 (1608 Metric), square (rectangular) end terminal, IPC-7351 nominal, (Body size source: http://www.tortai-tech.com/upload/download/2011102023233369053.pdf), generated with kicad-footprint-generator")
 		(tags "LED handsolder")
@@
 	(footprint "Library:SOP65P640X120-20N"
 		(layer "F.Cu")
-		(at 150.5 58)
+		(at 119.8 60.8)
 		(property "Reference" "U4"
 			(at -0.325 -4.385 0)
@@
 		)
 		(embedded_fonts no)
+		(model "${KIPRJMOD}/lib/PCM5102APWR/PCM5102APWR.step"
+			(offset
+				(xyz 0 0 0)
+			)
+			(scale
+				(xyz 1 1 1)
+			)
+			(rotate
+				(xyz -90 -0 -0)
+			)
+		)
 	)
 	(footprint "Capacitor_SMD:C_0603_1608Metric_Pad1.08x0.95mm_HandSolder"
@@
 	(footprint "Library:MJ-8435"
 		(layer "F.Cu")
-		(at 141.5 79.5 180)
+		(at 129 80.3 180)
 		(descr "MJ-8435")
 		(tags "Connector")

Commit message: update11
Parts:
- added R26: 100kΩ, Resistor_SMD:R_0603_1608Metric_Pad0.98x0.95mm_HandSolder, F.Cu at (88.6, 92.0)
- added R27: 100kΩ, Resistor_SMD:R_0603_1608Metric_Pad0.98x0.95mm_HandSolder, F.Cu at (88.6, 94.5)
- moved FB1 94.2 mm to (154.8, 17.0)
- moved U2 86.4 mm to (116.3, 28.5)
- moved Q1 84.3 mm to (130.5, 46.5)
- moved SW1 82.9 mm to (188.0, 44.5)
- moved VR1 76.9 mm to (130.5, 43.0)
- moved U1 73.5 mm to (125.5, 20.5), turned to -90 degrees
- moved D5 62.2 mm to (160.5, 84.1), turned to -90 degrees
- moved U7 62.2 mm to (145.5, 39.5)
- moved D6 59.1 mm to (157.9, 84.1), turned to -90 degrees
- moved D7 56.0 mm to (155.3, 84.1), turned to -90 degrees
- moved SW6 52.3 mm to (171.0, 27.5), turned to -90 degrees
- moved R25 52.1 mm to (81.1, 65.0)
- moved D4 48.2 mm to (127.5, 43.1), turned to 90 degrees
- moved D3 42.9 mm to (127.5, 46.6), turned to -90 degrees
- moved U3 40.9 mm to (197.2, 81.9)
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Connections:
- U3 pad 11: unconnected-(U3-IO18-Pad11) -> BTN_3
- U3 pad 12: BTN_3 -> Net-(U3-IO8)

Commit message: update
Parts:
- removed C34: 10μF, Capacitor_SMD:C_0603_1608Metric_Pad1.08x0.95mm_HandSolder
- removed D5, D6, D7: LED, LED_SMD:LED_0603_1608Metric_Pad1.05x0.95mm_HandSolder
- removed Q1: MMBT3904, Library:TRANS_MMBT3904
- removed R19: 10kΩ, Resistor_SMD:R_0603_1608Metric_Pad0.98x0.95mm_HandSolder
- removed R23: 1kΩ, Resistor_SMD:R_0603_1608Metric_Pad0.98x0.95mm_HandSolder
- removed R24: 47Ω, Resistor_SMD:R_0603_1608Metric_Pad0.98x0.95mm_HandSolder
- removed SW4: ENC_SW, Button_Switch_THT:SW_Tactile_SPST_Angled_PTS645Vx39-2LFS
- moved J3 125.1 mm to (242.0, 61.6)
- moved R5 101.6 mm to (172.0, 34.0)
- moved R4 97.1 mm to (168.2, 34.0), turned to 180 degrees
- moved SW7 93.7 mm to (212.0, 42.8), turned to -90 degrees
- moved J5 83.3 mm to (272.3, 69.5), turned to 90 degrees
- moved D2 83.0 mm to (172.0, 31.5)
- moved R3 79.4 mm to (156.5, 45.0), turned to -90 degrees
- moved D1 78.4 mm to (168.1, 31.5)
- moved C22 67.2 mm to (170.9, 47.6), turned to 180 degrees
- moved C20 66.9 mm to (171.8, 57.0), turned to 180 degrees
- moved C19 58.8 mm to (166.0, 44.2), turned to 90 degrees
- moved U5 58.5 mm to (169.9, 41.8), turned to -90 degrees
- moved S1 57.6 mm to (145.0, 74.0)
- moved C18 56.1 mm to (164.0, 44.2), turned to -90 degrees
- moved SW5 54.0 mm to (202.0, 42.8)
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Connections:
- C4 pad 1: Net-(SW1-A) -> Net-(SW1-C)
- SW1 pad 1: Net-(SW1-A) -> unconnected-(SW1-A-Pad1)
- SW1 pad 3: unconnected-(SW1-C-Pad3) -> Net-(SW1-C)
- U3 pad 15: ENC_SW -> unconnected-(U3-IO3-Pad15)
- U3 pad 4: LED -> unconnected-(U3-IO4-Pad4)
- VR1 pad 3: Net-(SW1-A) -> Net-(SW1-C)
Routing:
- net Out_L: track 0.00 -> 34.0 mm, vias 0 -> 1
- net +3.3V: track 0.00 -> 31.9 mm
- net Out_R: track 0.00 -> 23.4 mm, vias 0 -> 1
- net Net-(U2-STAT): track 0.00 -> 19.4 mm, vias 0 -> 2
- net VBUS_FILT: track 0.00 -> 14.2 mm
- net VBAT: track 0.00 -> 11.2 mm
- net Net-(FB1-Pad2): track 0.00 -> 10.8 mm
- net Net-(D3-K): track 0.00 -> 9.31 mm
- net Net-(SW1-C): track 0.00 -> 7.90 mm
- net I2S_BCLK: track 0.00 -> 7.35 mm, vias 0 -> 2
- net USB_DP: track 0.00 -> 7.14 mm
- net USB_DM: track 0.00 -> 6.44 mm
- net AUDIO_L: track 0.00 -> 5.59 mm
- net AUDIO_R: track 0.00 -> 4.86 mm
- net I2S_LRCK: track 0.00 -> 4.71 mm
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Other:
- board size 48 x 58 mm -> 148 x 58 mm

Commit message: update
Parts:
- moved R8 130.7 mm to (241.2, 81.0)
- moved C9 118.2 mm to (239.2, 62.9), turned to -90 degrees
- moved R2 87.1 mm to (162.3, 37.4)
- moved R1 81.7 mm to (157.5, 37.5)
- moved R27 81.5 mm to (161.2, 57.5)
- moved R26 81.0 mm to (161.2, 56.0), turned to 180 degrees
- moved C1 71.3 mm to (155.9, 40.5), turned to 90 degrees
- moved C30 61.5 mm to (139.1, 57.9), turned to 180 degrees
- moved C31 56.0 mm to (139.1, 56.4), turned to 180 degrees
- moved S2 2.00 mm to (152.1, 76.0)
- moved S1 2.00 mm to (145.0, 76.0)
Routing:
- net +3.3V: track 31.9 -> 86.5 mm, vias 0 -> 5
- net GND: track 0.00 -> 49.4 mm, vias 0 -> 4
- net ENC_B: track 0.00 -> 35.2 mm, vias 0 -> 1
- net Net-(U3-EN): track 0.00 -> 34.7 mm, vias 0 -> 2
- net VDD_1.9V: track 0.00 -> 33.2 mm, vias 0 -> 1
- net ENC_A: track 0.00 -> 32.3 mm, vias 0 -> 1
- net Net-(U3-IO0): track 0.00 -> 17.5 mm
- net OPT_CS: track 0.00 -> 15.8 mm, vias 0 -> 2
- net VBAT: track 11.2 -> 20.2 mm
- net OPT_MISO: track 0.00 -> 8.12 mm
- net SDA: track 0.00 -> 7.39 mm
- net SCL: track 0.00 -> 6.61 mm
- net Net-(U6-VDDPIX): track 0.00 -> 4.44 mm
- net Net-(U3-IO8): track 0.00 -> 3.61 mm
- net Net-(U2-STAT): track 19.4 -> 21.6 mm
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- added copper zone on B.Cu, net GND
- added copper zone on F.Cu, net GND
Other:
- outline, holes or cut-outs redrawn

Commit message: update
Parts:
- added J2: Connector, Connector_PinSocket_2.00mm:PinSocket_1x17_P2.00mm_Vertical, F.Cu at (176.0, 80.7)
- moved R25 182.2 mm to (273.8, 75.7)
- moved C23 179.3 mm to (257.6, 67.9), turned to 180 degrees
- moved R12 173.6 mm to (260.9, 66.7)
- moved R14 173.4 mm to (260.9, 64.5)
- moved R9 173.3 mm to (256.5, 72.2)
- moved R13 170.1 mm to (257.6, 65.6)
- moved R11 169.6 mm to (256.5, 69.8)
- moved R10 166.7 mm to (253.3, 71.0)
- moved C36 141.2 mm to (222.9, 44.3), turned to 180 degrees
- moved R21 131.8 mm to (222.9, 45.8), turned to 180 degrees
- moved C37 130.3 mm to (211.4, 44.3), turned to 180 degrees
- moved R22 120.7 mm to (211.4, 45.8), turned to 180 degrees
- moved C35 118.1 mm to (199.8, 44.3), turned to 180 degrees
- moved R20 108.6 mm to (199.8, 45.8), turned to 180 degrees
- moved C33 96.5 mm to (179.6, 52.4)
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Routing:
- net +3.3V: track 86.5 -> 160.8 mm
- net BTN_3: track 0.00 -> 29.2 mm, vias 0 -> 1
- net BTN_1: track 0.00 -> 28.7 mm, vias 0 -> 1
- net BTN_2: track 0.00 -> 28.2 mm, vias 0 -> 1
- net LCD_RES: track 0.00 -> 24.0 mm, vias 0 -> 1
- net LCD_BLK: track 0.00 -> 23.3 mm, vias 0 -> 1
- net LCD_DC: track 0.00 -> 22.7 mm, vias 0 -> 1
- net USB_DM_PROT: track 0.00 -> 21.9 mm, vias 0 -> 2
- net SD_CD: track 0.00 -> 20.9 mm, vias 0 -> 1
- net USB_DP_PROT: track 0.00 -> 20.5 mm, vias 0 -> 2
- net SDA: track 7.39 -> 27.7 mm, vias 0 -> 1
- net SCL: track 6.61 -> 26.5 mm, vias 0 -> 1
- net ENC_B: track 35.2 -> 49.0 mm
- net ENC_A: track 32.3 -> 40.9 mm
- net SD_DAT3: track 0.00 -> 4.82 mm
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Other:
- outline, holes or cut-outs redrawn
