File: PocketNode_kicad/PocketNode.kicad_pcb (KiCad board)
At the start: 2 copper layers, 148 x 58 mm, 86 parts, among them J1 USB4105-GF-A, J2 Connector, J3 display, J4 MJ-8435, J5 DM3AT-SF-PEJM5, SW1 Power, SW5 SW1, SW6 SW2, SW7 SW3, U1 USBLC6-2SC6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

Commit message: update
Parts:
- added C38: 0.1μF, Capacitor_SMD:C_0603_1608Metric_Pad1.08x0.95mm_HandSolder, F.Cu at (1.68, 0.76)
- J2: footprint Connector_PinSocket_2.00mm:PinSocket_1x17_P2.00mm_Vertical -> Connector_PinSocket_2.00mm:PinSocket_1x17_P2.00mm_Horizontal
- moved J2 32.1 mm to (144.0, 79.6), turned to 90 degrees
Connections:
- J2 pad 1: +3.3V -> SCL
- J2 pad 10: BTN_2 -> SD_CMD
- J2 pad 11: BTN_1 -> SD_DAT0
- J2 pad 12: BTN_3 -> SD_DAT1
- J2 pad 13: LCD_RES -> SD_DAT2
- J2 pad 14: LCD_BLK -> SD_DAT3
- J2 pad 15: LCD_DC -> SD_CD
- J2 pad 16: SDA -> GND
- J2 pad 17: SCL -> +3.3V
- J2 pad 2: GND -> SDA
- J2 pad 3: SD_CD -> LCD_DC
- J2 pad 4: SD_DAT3 -> LCD_BLK
- J2 pad 5: SD_DAT2 -> LCD_RES
- J2 pad 6: SD_DAT1 -> BTN_3
- J2 pad 7: SD_DAT0 -> BTN_1
- J2 pad 8: SD_CMD -> BTN_2
Routing:
- net SD_DAT0: track 3.91 -> 2.79 mm
- net SD_DAT1: track 4.21 -> 3.09 mm
- net SD_DAT2: track 4.51 -> 3.39 mm
- net SD_CMD: track 3.64 -> 2.56 mm
- net SD_CLK: track 3.95 -> 2.87 mm
- net BTN_2: track 28.2 -> 27.1 mm
- net BTN_1: track 28.7 -> 27.6 mm
- net +3.3V: track 160.8 -> 159.8 mm
- net SD_CD: track 20.9 -> 19.8 mm
- net BTN_3: track 29.2 -> 28.5 mm
- net SD_DAT3: track 4.82 -> 4.19 mm

Commit message: update
Parts:
- added J6: Connector, Connector_PinSocket_2.00mm:PinSocket_1x17_P2.00mm_Horizontal, F.Cu at (194.0, 79.7)
- added J7: Connector, Connector_PinSocket_2.00mm:PinSocket_1x17_P2.00mm_Horizontal, F.Cu at (244.0, 79.7)
- moved C38 157.3 mm to (142.0, 71.8), turned to 180 degrees
- moved R14 4.10 mm to (257.0, 63.4)
- moved R12 3.96 mm to (257.0, 66.3)
- moved R10 3.72 mm to (257.0, 70.8)
- moved R13 0.98 mm to (257.0, 64.8)
- moved R11 0.66 mm to (257.0, 69.3)
- moved C23 0.59 mm to (257.0, 67.8)
- moved R9 0.50 mm to (257.0, 72.3)
Routing:
- net +3.3V: track 159.8 -> 317.0 mm, vias 5 -> 8
- net BTN_2: track 27.1 -> 99.0 mm
- net BTN_3: track 28.5 -> 90.1 mm, vias 1 -> 3
- net BTN_1: track 27.6 -> 75.8 mm
- net SD_DAT2: track 3.39 -> 27.5 mm, vias 0 -> 1
- net SD_DAT3: track 4.19 -> 28.0 mm, vias 0 -> 2
- net SD_CMD: track 2.56 -> 22.4 mm, vias 0 -> 1
- net SCL: track 26.1 -> 44.8 mm
- net SD_CLK: track 2.87 -> 20.7 mm, vias 0 -> 1
- net SDA: track 27.3 -> 44.8 mm
- net SD_DAT0: track 2.79 -> 20.0 mm, vias 0 -> 1
- net SD_DAT1: track 3.09 -> 18.5 mm, vias 0 -> 1
- net LCD_RES: track 23.6 -> 37.8 mm
- net LCD_DC: track 22.3 -> 32.3 mm
- net LCD_BLK: track 22.9 -> 29.7 mm
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Other:
- outline, holes or cut-outs redrawn
