File: PocketNode_kicad/LED.kicad_sch (KiCad schematic)
At the start: 6 parts, among them Q1 MMBT3904

Commit message: update
Parts:
- D5, D6, D7: footprint (none) -> LED_SMD:LED_0603_1608Metric_Pad1.05x0.95mm_HandSolder
- Q1: footprint MMBT3904 -> Library:TRANS_MMBT3904
- R23: footprint (none) -> Resistor_SMD:R_0603_1608Metric_Pad0.98x0.95mm_HandSolder
- R24: value 100Ω -> 47Ω; footprint (none) -> Resistor_SMD:R_0603_1608Metric_Pad0.98x0.95mm_HandSolder
Changed lines of the file:
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@@
 			)
 		)
-		(property "Footprint" ""
+		(property "Footprint" "LED_SMD:LED_0603_1608Metric_Pad1.05x0.95mm_HandSolder"
 			(at 130.81 63.5 0)
 			(effects
@@
 			)
 		)
-		(property "Value" "100Ω"
+		(property "Value" "47Ω"
 			(at 140.97 58.4199 0)
 			(effects
@@
 			)
 		)
-		(property "Footprint" ""
+		(property "Footprint" "Resistor_SMD:R_0603_1608Metric_Pad0.98x0.95mm_HandSolder"
 			(at 138.43 57.15 0)
 			(effects
@@
 			)
 		)
-		(property "Footprint" "MMBT3904"
+		(property "Footprint" "Library:TRANS_MMBT3904"
 			(at 135.89 80.01 0)
 			(effects
@@
 			)
 		)
-		(property "Footprint" ""
+		(property "Footprint" "LED_SMD:LED_0603_1608Metric_Pad1.05x0.95mm_HandSolder"
 			(at 138.43 63.5 0)
 			(effects
@@
 			)
 		)
-		(property "Footprint" ""
+		(property "Footprint" "LED_SMD:LED_0603_1608Metric_Pad1.05x0.95mm_HandSolder"
 			(at 146.05 63.5 0)
 			(effects
@@
 			)
 		)
-		(property "Footprint" ""
+		(property "Footprint" "Resistor_SMD:R_0603_1608Metric_Pad0.98x0.95mm_HandSolder"
 			(at 130.81 80.01 0)
 			(effects

Commit message: update
Parts:
- removed D5, D6, D7: LED, LED_SMD:LED_0603_1608Metric_Pad1.05x0.95mm_HandSolder, symbol Device:LED
- removed Q1: MMBT3904, Library:TRANS_MMBT3904, symbol Library:MMBT3904
- removed R23: 1kΩ, Resistor_SMD:R_0603_1608Metric_Pad0.98x0.95mm_HandSolder, symbol Device:R_Small
- removed R24: 47Ω, Resistor_SMD:R_0603_1608Metric_Pad0.98x0.95mm_HandSolder, symbol Device:R_Small
