File: PocketNode_kicad/power.kicad_sch (KiCad schematic)
At the start: 21 parts, among them J1 USB4105-GF-A, SW1 SW_SPDT, U1 USBLC6-2SC6, U2 MCP73831T-2ACI_OT

Commit message: update2
Parts:
- C5: value 1μF -> 10μF
- SW1: value SW_SPDT -> Power
Changed lines of the file:
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@@
 	(wire
 		(pts
-			(xy 120.65 92.71) (xy 114.3 92.71)
+			(xy 121.92 92.71) (xy 114.3 92.71)
 		)
 		(stroke
@@
 	(global_label "+3.3V"
 		(shape input)
-		(at 120.65 92.71 0)
+		(at 121.92 92.71 0)
 		(fields_autoplaced yes)
 		(effects
@@
 		)
 		(property "Intersheetrefs" "${INTERSHEET_REFS}"
-			(at 129.32 92.71 0)
+			(at 130.59 92.71 0)
 			(effects
 				(font
@@
 			)
 		)
-		(property "Value" "SW_SPDT"
+		(property "Value" "Power"
 			(at 60.96 88.9 0)
 			(effects
@@
 			)
 		)
-		(property "Value" "1μF"
+		(property "Value" "10μF"
 			(at 116.84 91.4335 0)
 			(effects

Commit message: update
Parts:
- C1, C2, C3, C4, C5: footprint (none) -> Capacitor_SMD:C_0603_1608Metric_Pad1.08x0.95mm_HandSolder
- D1, D2: footprint (none) -> LED_SMD:LED_0603_1608Metric_Pad1.05x0.95mm_HandSolder
- D3, D4: footprint (none) -> Diode_SMD:D_0603_1608Metric_Pad1.05x0.95mm_HandSolder
- J1: footprint USB4105-GF-A -> Library:GCT_USB4105-GF-A
- R1, R2, R3, R4, R5: footprint (none) -> Resistor_SMD:R_0603_1608Metric_Pad0.98x0.95mm_HandSolder
- U1: footprint USBLC6-2SC6 -> Library:SOT95P280X145-6N
- U2: footprint MCP73831T-2ACI_OT -> Library:SOT95P280X145-5N
- VR1: footprint MCP1700T-3302E_TT -> Library:SOT95P237X112-3N
Changed lines of the file:
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@@
 			)
 		)
-		(property "Footprint" "MCP1700T-3302E_TT"
+		(property "Footprint" "Library:SOT95P237X112-3N"
 			(at 93.98 95.25 0)
 			(effects
@@
 			)
 		)
-		(property "Footprint" ""
+		(property "Footprint" "Capacitor_SMD:C_0603_1608Metric_Pad1.08x0.95mm_HandSolder"
 			(at 97.79 73.66 0)
 			(effects
@@
 			)
 		)
-		(property "Footprint" ""
+		(property "Footprint" "Capacitor_SMD:C_0603_1608Metric_Pad1.08x0.95mm_HandSolder"
 			(at 168.91 36.83 0)
 			(effects
@@
 			)
 		)
-		(property "Footprint" ""
+		(property "Footprint" "Diode_SMD:D_0603_1608Metric_Pad1.05x0.95mm_HandSolder"
 			(at 40.64 92.71 90)
 			(effects
@@
 			)
 		)
-		(property "Footprint" "MCP73831T-2ACI_OT"
+		(property "Footprint" "Library:SOT95P280X145-5N"
 			(at 76.2 68.58 0)
 			(effects
@@
 			)
 		)
-		(property "Footprint" ""
+		(property "Footprint" "Diode_SMD:D_0603_1608Metric_Pad1.05x0.95mm_HandSolder"
 			(at 40.64 101.6 90)
 			(effects
@@
 			)
 		)
-		(property "Footprint" ""
+		(property "Footprint" "Resistor_SMD:R_0603_1608Metric_Pad0.98x0.95mm_HandSolder"
 			(at 87.63 31.75 0)
 			(effects
@@
 			)
 		)
-		(property "Footprint" ""
+		(property "Footprint" "Resistor_SMD:R_0603_1608Metric_Pad0.98x0.95mm_HandSolder"
 			(at 55.88 71.12 0)
 			(effects
@@
 			)
 		)
-		(property "Footprint" ""
+		(property "Footprint" "Resistor_SMD:R_0603_1608Metric_Pad0.98x0.95mm_HandSolder"
 			(at 34.29 31.75 0)
 			(effects
@@
 			)
 		)
-		(property "Footprint" ""
+		(property "Footprint" "Capacitor_SMD:C_0603_1608Metric_Pad1.08x0.95mm_HandSolder"
 			(at 38.1 68.58 0)
 			(effects
@@
 			)
 		)
-		(property "Footprint" ""
+		(property "Footprint" "Resistor_SMD:R_0603_1608Metric_Pad0.98x0.95mm_HandSolder"
 			(at 104.14 57.15 0)
 			(effects
@@
 			)
 		)
-		(property "Footprint" ""
+		(property "Footprint" "LED_SMD:LED_0603_1608Metric_Pad1.05x0.95mm_HandSolder"
 			(at 113.03 66.04 90)
 			(effects
@@
 			)
 		)
-		(property "Footprint" ""
+		(property "Footprint" "Capacitor_SMD:C_0603_1608Metric_Pad1.08x0.95mm_HandSolder"
 			(at 114.3 90.17 0)
 			(effects
@@
 			)
 		)
-		(property "Footprint" "USBLC6-2SC6"
+		(property "Footprint" "Library:SOT95P280X145-6N"
 			(at 146.05 34.29 0)
 			(effects
@@
 			)
 		)
-		(property "Footprint" ""
+		(property "Footprint" "LED_SMD:LED_0603_1608Metric_Pad1.05x0.95mm_HandSolder"
 			(at 113.03 57.15 90)
 			(effects
@@
 			)
 		)
-		(property "Footprint" ""
+		(property "Footprint" "Resistor_SMD:R_0603_1608Metric_Pad0.98x0.95mm_HandSolder"
 			(at 104.14 66.04 0)
 			(effects
@@
 			)
 		)
-		(property "Footprint" "USB4105-GF-A"
+		(property "Footprint" "Library:GCT_USB4105-GF-A"
 			(at 57.15 36.83 0)
 			(effects
@@
 			)
 		)
-		(property "Footprint" ""
+		(property "Footprint" "Capacitor_SMD:C_0603_1608Metric_Pad1.08x0.95mm_HandSolder"
 			(at 71.12 95.25 0)
 			(effects

Commit message: update
Parts:
- BT1: footprint (none) -> Connector_PinHeader_2.54mm:PinHeader_1x02_P2.54mm_Vertical
- FB1: value 100Ω@100MHz -> 120Ω@100MHz; footprint (none) -> Library:BEADC1608X95N
Changed lines of the file:
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@@
 			)
 		)
-		(property "Value" "100Ω@100MHz"
+		(property "Value" "120Ω@100MHz"
 			(at 92.7481 20.32 90)
 			(effects
@@
 			)
 		)
-		(property "Footprint" ""
+		(property "Footprint" "Library:BEADC1608X95N"
 			(at 92.71 22.352 90)
 			(effects
@@
 			)
 		)
-		(property "Footprint" ""
+		(property "Footprint" "Connector_PinHeader_2.54mm:PinHeader_1x02_P2.54mm_Vertical"
 			(at 142.24 75.946 90)
 			(effects

Commit message: update
Parts:
- SW1: footprint (none) -> Button_Switch_THT:SW_Slide_SPDT_Angled_CK_OS102011MA1Q
Changed lines of the file:
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@@
 			)
 		)
-		(property "Footprint" ""
+		(property "Footprint" "Button_Switch_THT:SW_Slide_SPDT_Angled_CK_OS102011MA1Q"
 			(at 60.96 95.25 0)
 			(effects

Commit message: update
Connections:
- net at C4.1, VR1.3 (VIN): now also SW1.3 (C); no longer SW1.1 (A)
Changed lines of the file:
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@@
+	)
+	(junction
+		(at 71.12 92.71)
+		(diameter 0)
+		(color 0 0 0 0)
 	)
 	(junction
@@
 		(color 0 0 0 0)
 	)
-	(junction
-		(at 71.12 92.71)
-		(diameter 0)
-		(color 0 0 0 0)
+	(no_connect
+		(at 66.04 92.71)
 	)
 	(no_connect
@@
 	)
 	(no_connect
-		(at 66.04 97.79)
-	)
-	(no_connect
 		(at 77.47 39.37)
 	)
 	(wire
 		(pts
+			(xy 66.04 95.25) (xy 68.58 95.25)
+		)
+		(stroke
+			(width 0)
+			(type default)
+		)
+	)
+	(wire
+		(pts
 			(xy 45.72 92.71) (xy 45.72 95.25)
 		)
@@
 	(wire
 		(pts
-			(xy 71.12 92.71) (xy 66.04 92.71)
-		)
-		(stroke
-			(width 0)
-			(type default)
-		)
-	)
-	(wire
-		(pts
 			(xy 106.68 66.04) (xy 110.49 66.04)
 		)
@@
 	(wire
 		(pts
+			(xy 68.58 95.25) (xy 68.58 92.71)
+		)
+		(stroke
+			(width 0)
+			(type default)
+		)
+	)
+	(wire
+		(pts
+			(xy 68.58 92.71) (xy 71.12 92.71)
+		)
+		(stroke
+			(width 0)
+			(type default)
+		)
+	)
+	(wire
+		(pts
 			(xy 45.72 101.6) (xy 43.18 101.6)
 		)
@@
 		)
 		(stroke
+			(width 0)
+			(type default)
+		)
+	)
+	(wire
+		(pts
+			(xy 66.04 97.79) (xy 66.04 95.25)
+		)
+		(stroke
