File: PocketNode_kicad/Sensors.kicad_sch (KiCad schematic)
At the start: 0 parts

Commit message: update4
Parts:
- added C23, C27, C29, C31: 0.1μF, symbol Device:C_Small
- added C24, C25: 1μF, symbol Device:C_Small
- added C26, C28: 10μF, symbol Device:C_Small
- added C30: 4.7μF, symbol Device:C_Small
- added J4: Micro_SD_Card_Det1, symbol Connector:Micro_SD_Card_Det1
- added R10, R11, R12, R13, R14, R9: 10kΩ, symbol Device:R_Small
- added R15: 52.3kΩ, symbol Device:R_Small
- added R16: 30.1kΩ, symbol Device:R_Small
- added U6: PMW3360DM-T2QU, symbol Library:PMW3360DM-T2QU
- added U7: TPS73601DBVR, TPS73601DBVR, symbol Library:TPS73601DBVR
Connections:
- new net: R15.1, R16.1, U7.4 (NR/FB)
- new net: C30.1, C31.1, U6.3 (VDDPIX)
- new net +3.3V: C23.1, C24.2, C28.1, C29.1, J4.4 (VDD), R10.1, R11.1, R12.1, R13.1, R14.1, R9.1, U6.5 (VDDIO), U7.1 (IN), U7.3 (EN)
- new net GND: C23.2, C24.1, C25.2, C26.2, C27.2, C28.2, C29.2, C30.2, C31.2, J4.10 (SHIELD), J4.6 (VSS), R16.2, U7.2 (GND)
- new net OPT_CS: U6.13 (~{CS})
- new net OPT_MISO: U6.12 (MISO)
- new net SCL: U6.10 (SCLK)
- new net SDA: U6.11 (MOSI)
- new net SD_CD: J4.9 (DET)
- new net SD_CLK: J4.5 (CLK), R11.2
- new net SD_CMD: J4.3 (CMD), R12.2
- new net SD_DAT0: J4.7 (DAT0), R10.2
- new net SD_DAT1: J4.8 (DAT1), R9.2
- new net SD_DAT2: J4.1 (DAT2), R14.2
- new net SD_DAT3: J4.2 (DAT3/CD), R13.2
- new net VDD_1.9V: C25.1, C26.1, C27.1, R15.2, U6.15 (LED_P), U6.4 (VDD), U7.5 (OUT)

Commit message: update5
Parts:
- added C32, C33, C34, C35, C36, C37: 10μF, symbol Device:C_Small
- added R17, R18, R19, R20, R21, R22: 10kΩ, symbol Device:R_Small
- added SW4: ENC_SW, symbol Switch:SW_Push
- added SW5: SW1, symbol Switch:SW_Push
- added SW6: SW2, symbol Switch:SW_Push
- added SW7: SW3, symbol Switch:SW_Push
- added VR2: EC10E, symbol Library:EC10E1220501
Connections:
- net +3.3V: now also U6.7 (~{RESET}), R17.2, R18.2, R19.2, R20.2, R21.2, R22.2
- net GND: now also U6.8 (GND), C32.2, C33.1, C34.2, C35.2, C36.2, C37.2, SW4.2, SW5.2, SW6.2, SW7.2, VR2.C
- new net BTN_1: C35.1, R20.1, SW5.1
- new net BTN_2: C36.1, R21.1, SW6.1
- new net BTN_3: C37.1, R22.1, SW7.1
- new net ENC_A: C33.2, R17.1, VR2.A
- new net ENC_B: C32.1, R18.1, VR2.B
- new net ENC_SW: C34.1, R19.1, SW4.1
- no-connect marks 0 -> 1

Commit message: update
Parts:
- C23, C24, C25, C26, C27, C28, C29, C30, C31, C32, C33, C34, C35, C36, C37: footprint (none) -> Capacitor_SMD:C_0603_1608Metric_Pad1.08x0.95mm_HandSolder
- R10, R11, R12, R13, R14, R15, R16, R17, R18, R19, R20, R21, R22, R9: footprint (none) -> Resistor_SMD:R_0603_1608Metric_Pad0.98x0.95mm_HandSolder
- U6: footprint (none) -> Library:PMW3360
- U7: footprint TPS73601DBVR -> Library:SOT95P280X145-5N
- VR2: footprint (none) -> Library:TRIM_EC10E1220501
Changed lines of the file:
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@@
 			)
 		)
-		(property "Footprint" ""
+		(property "Footprint" "Resistor_SMD:R_0603_1608Metric_Pad0.98x0.95mm_HandSolder"
 			(at 210.82 29.21 0)
 			(effects
@@
 			)
 		)
-		(property "Footprint" "TPS73601DBVR"
+		(property "Footprint" "Library:SOT95P280X145-5N"
 			(at 146.05 76.2 0)
 			(effects
@@
 			)
 		)
-		(property "Footprint" ""
+		(property "Footprint" "Capacitor_SMD:C_0603_1608Metric_Pad1.08x0.95mm_HandSolder"
 			(at 241.3 152.4 0)
 			(effects
@@
 			)
 		)
-		(property "Footprint" ""
+		(property "Footprint" "Resistor_SMD:R_0603_1608Metric_Pad0.98x0.95mm_HandSolder"
 			(at 229.87 149.86 0)
 			(effects
@@
 			)
 		)
-		(property "Footprint" ""
+		(property "Footprint" "Resistor_SMD:R_0603_1608Metric_Pad0.98x0.95mm_HandSolder"
 			(at 210.82 24.13 0)
 			(effects
@@
 			)
 		)
-		(property "Footprint" ""
+		(property "Footprint" "Resistor_SMD:R_0603_1608Metric_Pad0.98x0.95mm_HandSolder"
 			(at 210.82 34.29 0)
 			(effects
@@
 			)
 		)
-		(property "Footprint" ""
+		(property "Footprint" "Capacitor_SMD:C_0603_1608Metric_Pad1.08x0.95mm_HandSolder"
 			(at 250.19 66.04 0)
 			(effects
@@
 			)
 		)
-		(property "Footprint" ""
+		(property "Footprint" "Library:PMW3360"
 			(at 146.05 38.1 0)
 			(effects
@@
 			)
 		)
-		(property "Footprint" ""
+		(property "Footprint" "Resistor_SMD:R_0603_1608Metric_Pad0.98x0.95mm_HandSolder"
 			(at 231.14 71.12 0)
 			(effects
@@
 			)
 		)
-		(property "Footprint" ""
+		(property "Footprint" "Resistor_SMD:R_0603_1608Metric_Pad0.98x0.95mm_HandSolder"
 			(at 210.82 36.83 0)
 			(effects
@@
 			)
 		)
-		(property "Footprint" ""
+		(property "Footprint" "Capacitor_SMD:C_0603_1608Metric_Pad1.08x0.95mm_HandSolder"
 			(at 124.46 35.56 0)
 			(effects
@@
 			)
 		)
-		(property "Footprint" ""
+		(property "Footprint" "Capacitor_SMD:C_0603_1608Metric_Pad1.08x0.95mm_HandSolder"
 			(at 114.3 35.56 0)
 			(effects
@@
 			)
 		)
-		(property "Footprint" ""
+		(property "Footprint" "Capacitor_SMD:C_0603_1608Metric_Pad1.08x0.95mm_HandSolder"
 			(at 241.3 132.08 0)
 			(effects
@@
 			)
 		)
-		(property "Footprint" ""
+		(property "Footprint" "Resistor_SMD:R_0603_1608Metric_Pad0.98x0.95mm_HandSolder"
 			(at 123.19 76.2 0)
 			(effects
@@
 			)
 		)
-		(property "Footprint" ""
+		(property "Footprint" "Resistor_SMD:R_0603_1608Metric_Pad0.98x0.95mm_HandSolder"
 			(at 210.82 26.67 0)
 			(effects
@@
 			)
 		)
-		(property "Footprint" ""
+		(property "Footprint" "Capacitor_SMD:C_0603_1608Metric_Pad1.08x0.95mm_HandSolder"
 			(at 210.82 39.37 0)
 			(effects
@@
 			)
 		)
-		(property "Footprint" ""
+		(property "Footprint" "Capacitor_SMD:C_0603_1608Metric_Pad1.08x0.95mm_HandSolder"
 			(at 119.38 25.4 0)
 			(effects
@@
 			)
 		)
-		(property "Footprint" ""
+		(property "Footprint" "Capacitor_SMD:C_0603_1608Metric_Pad1.08x0.95mm_HandSolder"
 			(at 165.1 66.04 0)
 			(effects
@@
 			)
 		)
-		(property "Footprint" ""
+		(property "Footprint" "Resistor_SMD:R_0603_1608Metric_Pad0.98x0.95mm_HandSolder"
 			(at 229.87 110.49 0)
 			(effects
@@
 			)
 		)
-		(property "Footprint" ""
+		(property "Footprint" "Capacitor_SMD:C_0603_1608Metric_Pad1.08x0.95mm_HandSolder"
 			(at 242.57 73.66 0)
 			(effects
@@
 			)
 		)
-		(property "Footprint" ""
+		(property "Footprint" "Capacitor_SMD:C_0603_1608Metric_Pad1.08x0.95mm_HandSolder"
 			(at 104.14 33.02 0)
 			(effects
@@
 			)
 		)
-		(property "Footprint" ""
+		(property "Footprint" "Capacitor_SMD:C_0603_1608Metric_Pad1.08x0.95mm_HandSolder"
 			(at 241.3 113.03 0)
 			(effects
@@
 			)
 		)
-		(property "Footprint" ""
+		(property "Footprint" "Capacitor_SMD:C_0603_1608Metric_Pad1.08x0.95mm_HandSolder"
 			(at 93.98 33.02 0)
 			(effects
@@
 			)
 		)
-		(property "Footprint" ""
+		(property "Footprint" "Capacitor_SMD:C_0603_1608Metric_Pad1.08x0.95mm_HandSolder"
 			(at 241.3 92.71 0)
 			(effects
@@
 			)
 		)
-		(property "Footprint" ""
+		(property "Footprint" "Capacitor_SMD:C_0603_1608Metric_Pad1.08x0.95mm_HandSolder"
 			(at 104.14 73.66 0)
 			(effects
@@
 			)
 		)
-		(property "Footprint" ""
+		(property "Footprint" "Resistor_SMD:R_0603_1608Metric_Pad0.98x0.95mm_HandSolder"
 			(at 229.87 90.17 0)
 			(effects
@@
 			)
 		)
-		(property "Footprint" ""
+		(property "Footprint" "Resistor_SMD:R_0603_1608Metric_Pad0.98x0.95mm_HandSolder"
 			(at 238.76 68.58 0)
 			(effects
@@
 			)
 		)
-		(property "Footprint" ""
+		(property "Footprint" "Capacitor_SMD:C_0603_1608Metric_Pad1.08x0.95mm_HandSolder"
 			(at 109.22 25.4 0)
 			(effects
@@
 			)
 		)
-		(property "Footprint" ""
+		(property "Footprint" "Resistor_SMD:R_0603_1608Metric_Pad0.98x0.95mm_HandSolder"
 			(at 229.87 129.54 0)
 			(effects
@@
 			)
 		)
-		(property "Footprint" ""
+		(property "Footprint" "Resistor_SMD:R_0603_1608Metric_Pad0.98x0.95mm_HandSolder"
 			(at 210.82 31.75 0)
 			(effects
@@
 			)
 		)
-		(property "Footprint" ""
+		(property "Footprint" "Resistor_SMD:R_0603_1608Metric_Pad0.98x0.95mm_HandSolder"
 			(at 118.11 73.66 0)
 			(effects
@@
 			)
 		)
-		(property "Footprint" ""
+		(property "Footprint" "Library:TRIM_EC10E1220501"
 			(at 260.35 71.12 0)
 			(effects

Commit message: update
Parts:
- removed J4: Micro_SD_Card_Det1, symbol Connector:Micro_SD_Card_Det1
- added J5: DM3AT-SF-PEJM5, Library:HRS_DM3AT-SF-PEJM5, symbol Library:DM3AT-SF-PEJM5
- added R25: 10kΩ, Resistor_SMD:R_0603_1608Metric_Pad0.98x0.95mm_HandSolder, symbol Device:R_Small
Connections:
- net +3.3V: now also J5.4 (VDD), R25.1
- net GND: now also J5.6 (VSS), J5.P1 (SHIELD), J5.P2 (SHIELD), J5.P3 (SHIELD), J5.P4 (SHIELD), J5.SWB (B)
- net SD_CD: now also J5.SWA (A), R25.2
- net SD_CLK: now also J5.5 (CLK)
- net SD_CMD: now also J5.3 (CMD)
- net SD_DAT0: now also J5.7 (DAT0)
- net SD_DAT1: now also J5.8 (DAT1)
- net SD_DAT2: now also J5.1 (DAT2)
- net SD_DAT3: now also J5.2 (CD/DAT3)

Commit message: update
Parts:
- SW4: footprint (none) -> Button_Switch_THT:SW_Tactile_SPST_Angled_PTS645Vx39-2LFS
- SW5, SW6, SW7: footprint (none) -> Button_Switch_THT:SW_PUSH_6mm
Changed lines of the file:
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@@
 			)
 		)
-		(property "Footprint" ""
+		(property "Footprint" "Button_Switch_THT:SW_Tactile_SPST_Angled_PTS645Vx39-2LFS"
 			(at 252.73 85.09 0)
 			(effects
@@
 			)
 		)
-		(property "Footprint" ""
+		(property "Footprint" "Button_Switch_THT:SW_PUSH_6mm"
 			(at 252.73 144.78 0)
 			(effects
@@
 			)
 		)
-		(property "Footprint" ""
+		(property "Footprint" "Button_Switch_THT:SW_PUSH_6mm"
 			(at 252.73 124.46 0)
 			(effects
@@
 			)
 		)
-		(property "Footprint" ""
+		(property "Footprint" "Button_Switch_THT:SW_PUSH_6mm"
 			(at 252.73 105.41 0)
 			(effects

Commit message: update
Parts:
- removed C34: 10μF, Capacitor_SMD:C_0603_1608Metric_Pad1.08x0.95mm_HandSolder, symbol Device:C_Small
- removed R19: 10kΩ, Resistor_SMD:R_0603_1608Metric_Pad0.98x0.95mm_HandSolder, symbol Device:R_Small
- removed SW4: ENC_SW, Button_Switch_THT:SW_Tactile_SPST_Angled_PTS645Vx39-2LFS, symbol Switch:SW_Push
